Commit message: arrange pionner for ubuntu 14.04.

File: robots_description/pioneer_description/pioneer3at.xacro (robot description, xacro)
@@ -377,19 +377,4 @@
   </plugin>
 </gazebo>
- <joint name="tag_joint" type="fixed">
-    <axis xyz="0 0 0" />
-    <origin xyz="0 0 0.0" rpy="0 0 0"/>
-    <parent link="top_plate"/>
-    <child link="tag_link"/>
-  </joint>
-  <!-- april tag -->
-  <link name="tag_link">
-    <visual>
-      <origin xyz="0 0 0" rpy="0 0 0"/>
-      <geometry>
-        <mesh filename="model://april_tag_0/meshes/april_tag_0.dae"/>
-      </geometry>
-    </visual>
-  </link>
  <joint name="hokuyo_joint" type="fixed">
     <axis xyz="0 1 0" />
